File: kicad/kicad.sch (KiCad schematic (older format))
At the start: 26 parts

Commit message: Save progress on schematics.
Connections:
- net +5V: now also U?.12 (Q4), U?.12 (Q4), U?.14 (Q5), U?.14 (Q5), U?.14 (VCC), U?.14 (VCC), U?.14 (VCC), U?.16 (Q6), U?.16 (Q6), U?.18 (Q7), U?.20 (VCC), U?.20 (VCC), U?.24 (VCC), U?.3 (Q0), U?.5 (Q1), U?.7 (Q2), U?.9 (Q3)
- net GND: now also U?.10 (GND), U?.10 (GND), U?.12 (GND), U?.18 (*G1), U?.18 (Q7), U?.2 (P0), U?.3 (Q0), U?.4 (P1), U?.5 (Q1), U?.6 (P2), U?.7 (GND), U?.7 (GND), U?.7 (GND), U?.7 (Q2), U?.8 (P3), U?.9 (Q3)
- net at U?.17 (P7), U?.25 (A15), U?.9 (4A): now also U?.1 (1A)
- net at U?.2 (1Y), U?.22 (~OE): now also U?.2 (1B)
- net at U?.12 (6Y): now also U?.12 (4A)
- net at U?.3 (2A): now also U?.3 (1Y)
- net at U?.5 (3A): now also U?.11 (4Y), U?.19 (*G2)
- net at U?.6 (3Y): now also U?.2 (1B)
- net at U?.19 (*P=Q): now also U?.12 (4A)
- net at U?.19 (*P=Q): now also U?.13 (4B)
- net at U?.1 (0): now also U?.1 (OE)
- net at U?.2 (1): now also U?.1 (OE)
- net at U?.3 (2): now also U?.1 (OE)
- net at U?.4 (3): now also U?.13 (4B)
- net at U?.11 (4Y): now also U?.11 (Cp)

Commit message: Save progress on schematics.
Parts:
- removed U?: SN74HC32N, DIP794W45P254L1969H508Q14, symbol SN74HC32N:SN74HC32N
- J?: value Conn_01x13_Male -> Data In
Connections:
- net +5V: now also U?.14 (VCC), U?.20 (VCC), U?.20 (VCC), U?.20 (VCC)
- net GND: now also U?.10 (GND), U?.10 (GND), U?.10 (GND), U?.7 (GND)
- net at U?.19 (D7), U?.19 (D7), U?.19 (O7)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: now also U?.19 (O7), U?.19 (O7)
- net at U?.16 (O6), U?.18 (D6), U?.18 (D6)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: now also U?.16 (O6), U?.16 (O6)
- net at U?.15 (O5), U?.17 (D5), U?.17 (D5)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: now also U?.15 (O5), U?.15 (O5)
- net at U?.12 (O4), U?.16 (D4), U?.16 (D4)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: now also U?.12 (O4), U?.12 (O4)
- net at U?.15 (D3), U?.15 (D3), U?.30 (D3)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: now also U?.9 (O3), U?.9 (O3)
- net at U?.13 (D2), U?.13 (D2), U?.31 (D2)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: now also U?.6 (O2), U?.6 (O2)
- net at U?.12 (D1), U?.12 (D1), U?.32 (D1)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: now also U?.5 (O1), U?.5 (O1)
- net at U?.11 (D0), U?.11 (D0), U?.2 (O0)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: now also U?.2 (O0), U?.2 (O0)
- net at U?.12 (4A), U?.12 (6Y): now also U?.1 (1A), U?.4 (2A), U?.5 (2B), U?.9 (3A)
- net at U?.4 (2A): now also U?.8 (7)
- net at U?.6 (2Y): now also U?.11 (Cp) (x2)
- net at U?.5 (4): now also U?.10 (3B)
- net at U?.6 (5): now also U?.5 (2B)
- net at U?.7 (6): now also U?.2 (1B)
- net at U?.11 (Cp): now also J?.11 (Pin_11)
- net at U?.13 (D4): now also J?.4 (Pin_4), U?.13 (D4), U?.13 (D4)
- net at U?.14 (D5): now also J?.3 (Pin_3), U?.14 (D5), U?.14 (D5)
- net at U?.17 (D6): now also J?.2 (Pin_2), U?.17 (D6), U?.17 (D6)
- net at U?.18 (D7): now also J?.1 (Pin_1), U?.18 (D7), U?.18 (D7)
- net at U?.3 (D0): now also J?.8 (Pin_8), U?.3 (D0), U?.3 (D0)
- net at U?.4 (D1): now also J?.7 (Pin_7), U?.4 (D1), U?.4 (D1)
- net at U?.7 (D2): now also J?.6 (Pin_6), U?.7 (D2), U?.7 (D2)
- net at U?.8 (D3): now also J?.5 (Pin_5), U?.8 (D3), U?.8 (D3)
- net at U?.11 (Cp): now also J?.10 (Pin_10)
- net at U?.11 (Cp): now also J?.9 (Pin_9)
- net at U?.3 (1Y): now also U?.11 (Cp)
- net at U?.8 (3Y): now also U?.11 (Cp)

Commit message: Save progress on schematics.
Parts:
- added C? (x2): CP, symbol Device:CP
- added C? (x3): C, symbol Device:C
- added J?: Address Out, symbol Connector:Conn_01x18_Male
- added J?: Data Out, symbol Connector:Conn_01x05_Male
- added J?: Mode Out, symbol Connector:Conn_01x02_Male
- added J?: Power, symbol Connector:Conn_01x05_Male
Connections:
- net +5V: now also U?.20 (VCC), U?.20 (VCC), U?.20 (VCC), U?.20 (VCC), U?.20 (VCC), C?.1, C?.1, C?.1, C?.1, C?.1, J?.1 (Pin_1), J?.2 (Pin_2)
- net GND: now also U?.1 (OE), U?.1 (OE), U?.1 (OE), U?.1 (OE), U?.1 (OE), U?.10 (GND), U?.10 (GND), U?.10 (GND), U?.10 (GND), U?.10 (GND), C?.2, C?.2, C?.2, C?.2, C?.2, J?.3 (Pin_3), J?.4 (Pin_4), J?.5 (Pin_5)
- net at U?.19 (D7), U?.19 (D7), U?.19 (O7)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: now also U?.18 (D7), U?.18 (D7), U?.18 (D7), U?.18 (D7), U?.18 (D7)
- net at U?.16 (O6), U?.16 (O6), U?.16 (O6)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: now also U?.17 (D6), U?.17 (D6), U?.17 (D6), U?.17 (D6), U?.17 (D6)
- net at U?.15 (O5), U?.15 (O5), U?.15 (O5)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: now also U?.14 (D5), U?.14 (D5), U?.14 (D5), U?.14 (D5), U?.14 (D5)
- net at U?.12 (O4), U?.12 (O4), U?.12 (O4)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: now also U?.13 (D4), U?.13 (D4), U?.13 (D4), U?.13 (D4), U?.13 (D4)
- net at U?.15 (D3), U?.15 (D3), U?.30 (D3)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: now also U?.8 (D3), U?.8 (D3), U?.8 (D3), U?.8 (D3), U?.8 (D3)
- net at U?.13 (D2), U?.13 (D2), U?.31 (D2)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: now also U?.7 (D2), U?.7 (D2), U?.7 (D2), U?.7 (D2), U?.7 (D2)
- net at U?.12 (D1), U?.12 (D1), U?.32 (D1)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: now also U?.4 (D1), U?.4 (D1), U?.4 (D1), U?.4 (D1), U?.4 (D1)
- net at U?.11 (D0), U?.11 (D0), U?.2 (O0)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: now also U?.3 (D0), U?.3 (D0), U?.3 (D0), U?.3 (D0), U?.3 (D0)
- net at U?.12 (O4): now also J?.5 (Pin_5) (x2)
- net at U?.15 (O5): now also J?.6 (Pin_6)
- net at U?.16 (O6): now also J?.7 (Pin_7)
- net at U?.19 (O7): now also J?.8 (Pin_8)
- net at U?.2 (O0): now also J?.1 (Pin_1) (x3)
- net at U?.5 (O1): now also J?.2 (Pin_2) (x3)
- net at U?.6 (O2): now also J?.3 (Pin_3) (x2)
- net at U?.9 (O3): now also J?.4 (Pin_4) (x2)
- net at U?.12 (O4): now also J?.13 (Pin_13)
- net at U?.15 (O5): now also J?.14 (Pin_14)
- net at U?.16 (O6): now also J?.15 (Pin_15)
- net at U?.19 (O7): now also J?.16 (Pin_16)
- net at U?.2 (O0): now also J?.9 (Pin_9)
- net at U?.5 (O1): now also J?.10 (Pin_10)
- net at U?.6 (O2): now also J?.11 (Pin_11)
- net at U?.9 (O3): now also J?.12 (Pin_12)
- net at U?.2 (O0): now also J?.17 (Pin_17)
- net at U?.5 (O1): now also J?.18 (Pin_18)
Other:
- note added: "5V"
- note added: "CE"
- note added: "G"
- note added: "WE"

Commit message: Save progress on schematics.
Parts:
- C1, C5: renamed from C?; footprint (none) -> Capacitor_THT:CP_Radial_D12.5mm_P7.50mm
- C2, C3, C4: renamed from C?; footprint (none) -> Capacitor_THT:C_Axial_L3.8mm_D2.6mm_P7.50mm_Horizontal
- J1: renamed from J?; footprint (none) -> Connector_PinHeader_2.54mm:PinHeader_1x13_P2.54mm_Horizontal
- J2, J4: renamed from J?; footprint (none) -> Connector_PinHeader_2.54mm:PinHeader_1x05_P2.54mm_Horizontal
- J3: renamed from J?; footprint (none) -> Connector_PinHeader_2.54mm:PinHeader_1x18_P2.54mm_Horizontal
- J5: renamed from J?; footprint (none) -> Connector_PinHeader_2.54mm:PinHeader_1x02_P2.54mm_Horizontal
- R1, R2, R3, R4: renamed from R?; footprint (none) -> Resistor_THT:R_Axial_DIN0207_L6.3mm_D2.5mm_P10.16mm_Horizontal
- SW1: renamed from SW?; footprint (none) -> Button_Switch_THT:SW_PUSH_6mm_H4.3mm
- U1, U12, U15, U2, U5, U6, U8, U9: renamed from U?; footprint (none) -> Socket:DIP_Socket-20_W4.3_W5.08_W7.62_W10.16_W10.9_3M_220-3342-00-0602J
- U10, U13: renamed from U?; footprint (none) -> Socket:DIP_Socket-28_W11.9_W12.7_W15.24_W17.78_W18.5_3M_228-1277-00-0602J
- U11, U16: renamed from U?; footprint N20 -> Socket:DIP_Socket-20_W4.3_W5.08_W7.62_W10.16_W10.9_3M_220-3342-00-0602J
- U14, U17, U3, U7: renamed from U?; footprint DIP794W45P254L1969H508Q14 -> Socket:DIP_Socket-14_W4.3_W5.08_W7.62_W10.16_W10.9_3M_214-3339-00-0602J
- U18: renamed from U?; footprint N24_TEX -> Socket:DIP_Socket-24_W11.9_W12.7_W15.24_W17.78_W18.5_3M_224-1275-00-0602J
- U4: renamed from U?; footprint (none) -> Socket:DIP_Socket-40_W11.9_W12.7_W15.24_W17.78_W18.5_3M_240-1280-00-0602J
- gave numbers to parts that had none: 1
