File: kicad/kicad.kicad_pcb (KiCad board)
At the start: 4 copper layers, 245.1 x 125.7 mm, 31 parts, among them J1 Data In, J2 Power, J3 Address Out, J4 Data Out, J5 Mode Out, SW1 SW_Push_Dual, U1 74LS374, U10 AS6C62256-70PCN, U11 SN74LS682N, U12 74LS374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

Commit message: Save progress on PCB.
Parts:
- moved R4 42.0 mm to (134.6, 61.6)
- moved R2 41.2 mm to (109.9, 73.0), turned to 270 degrees
- moved R3 35.5 mm to (137.2, 83.8)
- moved R1 29.6 mm to (117.5, 83.2), turned to 90 degrees
Routing:
- net Net-(R2-Pad2): track 0.00 -> 30.0 mm
- net Net-(U4-Pad37): track 0.00 -> 18.1 mm
- net Net-(R1-Pad1): track 0.00 -> 10.8 mm
- net Net-(R3-Pad1): track 0.00 -> 3.81 mm
- net Net-(R4-Pad1): track 0.00 -> 3.17 mm
Other:
- board size 245.1 x 125.7 mm -> 165.7 x 93.3 mm
- board text added: "5V"
- board text added: "G"
- board text added: "GND"

Commit message: Save progress on PCB.
Routing:
- net Net-(U1-Pad4): track 0.00 -> 391.4 mm, vias 0 -> 10
- net Net-(U1-Pad3): track 0.00 -> 370.3 mm, vias 0 -> 3
- net Net-(U1-Pad18): track 0.00 -> 345.1 mm, vias 0 -> 5
- net Net-(U11-Pad17): track 0.00 -> 340.7 mm, vias 0 -> 1
- net Net-(U10-Pad2): track 0.00 -> 273.7 mm, vias 0 -> 3
- net Net-(U10-Pad1): track 0.00 -> 239.1 mm, vias 0 -> 3
- net Net-(U1-Pad11): track 0.00 -> 222.6 mm, vias 0 -> 3
- net Net-(U10-Pad10): track 0.00 -> 213.0 mm, vias 0 -> 1
- net Net-(U10-Pad9): track 0.00 -> 205.2 mm, vias 0 -> 3
- net Net-(U14-Pad8): track 0.00 -> 203.2 mm, vias 0 -> 4
- net Net-(U13-Pad20): track 0.00 -> 194.6 mm, vias 0 -> 1
- net Net-(U10-Pad8): track 0.00 -> 188.4 mm, vias 0 -> 1
- net Net-(U10-Pad7): track 0.00 -> 181.5 mm, vias 0 -> 2
- net Net-(U14-Pad6): track 0.00 -> 167.3 mm, vias 0 -> 2
- net Net-(J1-Pad12): track 0.00 -> 133.4 mm, vias 0 -> 4
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
Commit message: Save progress on PCB.
Routing:
- net Net-(U1-Pad7): track 95.2 -> 406.8 mm, vias 2 -> 16
- net Net-(U1-Pad13): track 125.1 -> 339.9 mm, vias 4 -> 12
- net Net-(U1-Pad14): track 119.2 -> 332.3 mm, vias 2 -> 11
- net Net-(U1-Pad17): track 120.2 -> 315.8 mm, vias 2 -> 6
- net Net-(U17-Pad11): track 29.1 -> 155.3 mm, vias 0 -> 4
- net Net-(U14-Pad1): track 49.6 -> 174.2 mm, vias 0 -> 1
- net Net-(U17-Pad2): track 0.00 -> 116.9 mm, vias 0 -> 4
- net Net-(U10-Pad26): track 88.9 -> 151.0 mm, vias 0 -> 6
- net Net-(U15-Pad11): track 0.00 -> 57.4 mm, vias 0 -> 1
- net Net-(U16-Pad19): track 0.00 -> 54.0 mm, vias 0 -> 2
- net Net-(J5-Pad1): track 0.00 -> 39.8 mm
- net Net-(J5-Pad2): track 0.00 -> 32.6 mm
- net Net-(U3-Pad13): track 28.0 -> 59.8 mm, vias 0 -> 2
- net Net-(U11-Pad19): track 0.00 -> 31.1 mm, vias 0 -> 2
- net Net-(U10-Pad22): track 67.7 -> 93.1 mm
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